File: Shield Schematic.sch (EAGLE design)
At the start: 48 parts

Commit message: Add files via upload
Parts:
- removed F4: FUSESH22,5A, fuse:FUSESH22,5A
- removed IC: LM386M-1, linear:LM386M-1
- removed J1: (no value), con-jack:JACK-PLUG1
- removed JP1, JP11, JP12, JP13, JP14, JP2, JP23, JP24, JP25, JP26, JP27, JP31, JP32, JP33, JP34, JP35, JP36, JP4, JP5, JP6, JP7, JP8, JP9: (no value), adafruit:PINHD-1X1
- removed R2: 10K, resistor:R-US_M0805
- removed R3: 10K, pot:TRIM_US-3223G
- removed R6: (no value), resistor:R-US_VMTB60
- added B2: ARDUINO_UNO_R3_SHIELDBASIC, SparkFun-Boards:ARDUINO_UNO_R3_SHIELDBASIC
- added C5, C6, C7, C8: (no value), capacitor-wima:C2,5-3
- added IC1: LM386N-1, linear:LM386N-1
- added J2: POWER_JACK, SparkFun-Connectors:POWER_JACK
- added R10, R11, R12, R9: (no value), resistor:R-US_0207/7
- added U1: 03540001ZXGY, SamacSys_Parts:03540001ZXGY
- C1: value 1uF -> (none); device resistor:CPOL-US085CS-1AR -> capacitor-wima:C2,5-3
- C2: value 0.05uF -> (none); device resistor:CPOL-US085CS-1AR -> capacitor-wima:C2,5-3
- C3: value 10uF -> (none); device resistor:CPOL-US085CS-1AR -> capacitor-wima:C2,5-3
- C4: value 250uF -> (none); device resistor:CPOL-US085CS-1AR -> capacitor-wima:C2,5-3
- JP3: device adafruit:PINHD-1X1 -> adafruit:PINHD-1X3; IOPIN 6 -> (none)
- R1: value 10K -> (none); device pot:TRIM_US-3223G -> pot:TRIM_US-B25P
- R4, R5, R7, R8: device resistor:R-US_VMTB60 -> resistor:R-US_0207/7
Connections:
- removed net ARDUINO_RESET: JP32.1
- removed net N$2: JP17.3
- removed net N$28: C1.+, IC.BYPASS
- removed net N$29: C2.+, C4.+, IC.OUT
- removed net N$3: JP17.5
- removed net N$30: C3.-, IC.GAIN@2
- removed net N$31: IC.+IN, R1.S
- removed net N$32: C2.-, R2.2
- removed net N$33: IC.GAIN@1, R3.E
- removed net N$34: C3.+, R3.S
- removed net N$4: F4.1, J1.3
- removed net N$6: JP17.4
- removed net N$7: JP17.6
- removed net NC: JP12.1, JP13.1, JP14.1, JP33.1, JP35.1, JP36.1
- new net N$11: C8.2, IC1.GAIN@2
- new net N$12: C8.1, R1.E
- new net N$13: IC1.GAIN@1, R1.S
- new net N$5: C6.1, C7.2, IC1.OUT
- new net N$8: C6.2, R5.2
- new net N$9: C5.1, IC1.BYPASS
- new net POT_OUT: IC1.+IN, JP3.2
- net +12V: now also B2.VIN, IC1.VS, U1.2; no longer F4.2, IC.VS, JP11.1
- net +5V_SERVO: now also C1.2, C2.2, C3.2, C4.2
- net +5V_UNO: now also B2.5V, JP17.4, JP17.6, JP17.8, R7.1, R8.1; no longer JP6.1
- net ACTION_BUTTON: now also B2.A3, JP17.7, R12.2; no longer JP18.1, JP24.1, R7.2
- net GND: now also B2.GND@0, B2.GND@1, B2.GND@2, C1.1, C2.1, C3.1, C4.1, C5.2, IC1.-IN, IC1.GND, J2.GND, J2.GNDBREAK, JP3.3, R10.1, R11.1, R12.1, R9.1; no longer C1.-, IC.-IN, IC.GND, J1.1, J1.2, JP23.1, JP34.1, R1.A, R2.1, R6.1, R7.1, R8.1
- net N$1: now also J2.PWR, U1.1; no longer JP17.1
- net PLAYLIVE_SWITCH: now also B2.A1, JP17.3, R9.2; no longer JP8.1, R5.2
- net PLAYRECORDING_SWITCH: now also B2.A2, JP17.5, R11.2; no longer JP9.1, R6.2
- net RECORD_SWITCH: now also B2.A0, JP17.1, R10.2; no longer JP7.1, R4.2
- net RESET_BUTTON: now also B2.D8, R4.2; no longer JP25.1, R8.2
- net SCL: now also B2.SCL, R8.2; no longer JP27.1
- net SDA: now also B2.SDA, R7.2; no longer JP26.1
- net SERVO1: now also B2.*D5; no longer JP2.1
- net SERVO2: now also B2.*D6; no longer JP3.1
- net SERVO3: now also B2.*D9; no longer JP4.1
- net SERVO4: now also B2.*D10; no longer JP5.1
- net SPEAKER: now also C7.1; no longer C4.-
- net TONE_IN: now also B2.*D3, JP3.1; no longer JP1.1, JP31.1, R1.E
Other:
- note removed: "4V-12V"
- note removed: "Audio Power Amplifier with Controlled Gain"
- note removed: "Gain = 20 - 200"
- moved on the sheet: JP17, R1, R4, R5, R7, R8

Commit message: Add files via upload
Parts:
- removed VR1: (no value), mylibrary:LM1085IT
- added IC2: LM1085IT-5.0, SamacSys_Parts:LM1085IT-5.0
Connections:
- net +12V: now also IC2.VIN; no longer VR1.INPUT
- net +5V_SERVO: now also IC2.VOUT; no longer VR1.OUTPUT
- net +5V_UNO: now also JP18.6, JP18.8
- net GND: now also IC2.ADJ/GND; no longer VR1.GND/ADJ
- net RESET_BUTTON: now also JP18.1; no longer JP18.3
Changed lines of the file:
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@@
 <part name="JP10" library="adafruit" library_urn="urn:adsk.eagle:library:420" deviceset="PINHD-1X3" device="" package3d_urn="urn:adsk.eagle:package:6240710/1"/>
 <part name="JP15" library="adafruit" deviceset="PINHD-2X4" device=""/>
-<part name="VR1" library="mylibrary" deviceset="LM1085IT" device=""/>
 <part name="JP16" library="adafruit" deviceset="PINHD-2X4" device=""/>
 <part name="FRAME1" library="frames" library_urn="urn:adsk.eagle:library:229" deviceset="FRAME_C_L" device=""/>
@@
 <part name="J2" library="SparkFun-Connectors" library_urn="urn:adsk.eagle:library:513" deviceset="POWER_JACK" device="" package3d_urn="urn:adsk.eagle:package:38231/1"/>
 <part name="U1" library="SamacSys_Parts" deviceset="03540001ZXGY" device=""/>
+<part name="IC2" library="SamacSys_Parts" deviceset="LM1085IT-5.0" device=""/>
 </parts>
 <sheets>
@@
 <attribute name="VALUE" x="110.49" y="-5.08" size="1.778" layer="96"/>
 </instance>
-<instance part="VR1" gate="G$1" x="299.72" y="101.6" smashed="yes">
-<attribute name="NAME" x="299.72" y="119.38" size="1.778" layer="95"/>
-<attribute name="VALUE" x="302.26" y="99.06" size="1.778" layer="95"/>
-</instance>
 <instance part="JP16" gate="A" x="304.8" y="264.16" smashed="yes">
 <attribute name="NAME" x="298.45" y="272.415" size="1.778" layer="95"/>
@@
 <attribute name="NAME" x="328.93" y="152.4" size="1.778" layer="95" align="center-left"/>
 <attribute name="VALUE" x="328.93" y="149.86" size="1.778" layer="96" align="center-left"/>
+</instance>
+<instance part="IC2" gate="G$1" x="294.64" y="88.9" smashed="yes">
+<attribute name="NAME" x="318.77" y="96.52" size="1.778" layer="95" align="center-left"/>
+<attribute name="VALUE" x="318.77" y="93.98" size="1.778" layer="96" align="center-left"/>
 </instance>
 </instances>
@@
 <junction x="132.08" y="7.62"/>
 <label x="137.16" y="7.62" size="1.778" layer="95" xref="yes"/>
-</segment>
-<segment>
-<pinref part="VR1" gate="G$1" pin="GND/ADJ"/>
-<wire x1="294.64" y1="104.14" x2="289.56" y2="104.14" width="0.1524" layer="91"/>
-<label x="289.56" y="104.14" size="1.778" layer="95" rot="R180" xref="yes"/>
 </segment>
 <segment>
@@
 <label x="297.18" y="134.62" size="1.778" layer="95" xref="yes"/>
 </segment>
+<segment>
+<pinref part="IC2" gate="G$1" pin="ADJ/GND"/>
+<wire x1="294.64" y1="88.9" x2="294.64" y2="93.98" width="0.1524" layer="91"/>
+<wire x1="294.64" y1="93.98" x2="284.48" y2="93.98" width="0.1524" layer="91"/>
+<label x="284.48" y="93.98" size="1.778" layer="95" rot="R180" xref="yes"/>
+</segment>
 </net>
 <net name="SPEAKER" class="3">
@@
 </segment>
 <segment>
-<pinref part="JP18" gate="A" pin="3"/>
-<wire x1="284.48" y1="48.26" x2="279.4" y2="48.26" width="0.1524" layer="91"/>
-<wire x1="279.4" y1="48.26" x2="279.4" y2="45.72" width="0.1524" layer="91"/>
-<wire x1="279.4" y1="45.72" x2="274.32" y2="45.72" width="0.1524" layer="91"/>
-<label x="274.32" y="45.72" size="1.778" layer="95" rot="R180" xref="yes"/>
-</segment>
-<segment>
 <pinref part="B2" gate="G$1" pin="D8"/>
 <wire x1="116.84" y1="220.98" x2="134.62" y2="220.98" width="0.1524" layer="91"/>
@@
 <wire x1="134.62" y1="231.14" x2="147.32" y2="231.14" width="0.1524" layer="91"/>
 <label x="147.32" y="231.14" size="1.778" layer="95" xref="yes"/>
+</segment>
+<segment>
+<pinref part="JP18" gate="A" pin="1"/>
+<wire x1="284.48" y1="50.8" x2="274.32" y2="50.8" width="0.1524" layer="91"/>
+<label x="274.32" y="50.8" size="1.778" layer="95" rot="R180" xref="yes"/>
 </segment>
 </net>
@@
 <segment>
 <pinref part="JP18" gate="A" pin="2"/>
-<wire x1="292.1" y1="50.8" x2="302.26" y2="50.8" width="0.1524" layer="91"/>
+<wire x1="292.1" y1="50.8" x2="297.18" y2="50.8" width="0.1524" layer="91"/>
 <label x="302.26" y="50.8" size="1.778" layer="95" xref="yes"/>
-</segment>
-<segment>
 <pinref part="JP18" gate="A" pin="4"/>
-<wire x1="292.1" y1="48.26" x2="299.72" y2="48.26" width="0.1524" layer="91"/>
-<wire x1="299.72" y1="48.26" x2="299.72" y2="45.72" width="0.1524" layer="91"/>
-<wire x1="299.72" y1="45.72" x2="304.8" y2="45.72" width="0.1524" layer="91"/>
-<label x="304.8" y="45.72" size="1.778" layer="95" xref="yes"/>
+<wire x1="297.18" y1="50.8" x2="302.26" y2="50.8" width="0.1524" layer="91"/>
+<wire x1="292.1" y1="48.26" x2="297.18" y2="48.26" width="0.1524" layer="91"/>
+<wire x1="297.18" y1="48.26" x2="297.18" y2="50.8" width="0.1524" layer="91"/>
+<junction x="297.18" y="50.8"/>
+<pinref part="JP18" gate="A" pin="6"/>
+<wire x1="292.1" y1="45.72" x2="297.18" y2="45.72" width="0.1524" layer="91"/>
+<wire x1="297.18" y1="45.72" x2="297.18" y2="48.26" width="0.1524" layer="91"/>
+<junction x="297.18" y="48.26"/>
+<pinref part="JP18" gate="A" pin="8"/>
+<wire x1="292.1" y1="43.18" x2="297.18" y2="43.18" width="0.1524" layer="91"/>
+<wire x1="297.18" y1="43.18" x2="297.18" y2="45.72" width="0.1524" layer="91"/>
+<junction x="297.18" y="45.72"/>
 </segment>
 <segment>
@@
 <net name="+12V" class="2">
 <segment>
-<pinref part="VR1" gate="G$1" pin="INPUT"/>
-<wire x1="294.64" y1="114.3" x2="289.56" y2="114.3" width="0.1524" layer="91"/>
-<label x="289.56" y="114.3" size="1.778" layer="95" rot="R180" xref="yes"/>
-</segment>
-<segment>
 <pinref part="B2" gate="G$1" pin="VIN"/>
 <wire x1="91.44" y1="218.44" x2="76.2" y2="218.44" width="0.1524" layer="91"/>
@@
 <label x="327.66" y="137.16" size="1.778" layer="95" xref="yes"/>
 </segment>
+<segment>
+<pinref part="IC2" gate="G$1" pin="VIN"/>
+<wire x1="294.64" y1="83.82" x2="294.64" y2="78.74" width="0.1524" layer="91"/>
+<wire x1="294.64" y1="78.74" x2="284.48" y2="78.74" width="0.1524" layer="91"/>
+<label x="284.48" y="78.74" size="1.778" layer="95" rot="R180" xref="yes"/>
+</segment>
 </net>
 <net name="+5V_SERVO" class="2">
-<segment>
-<pinref part="VR1" gate="G$1" pin="OUTPUT"/>
-<wire x1="317.5" y1="109.22" x2="327.66" y2="109.22" width="0.1524" layer="91"/>
-<label x="327.66" y="109.22" size="1.778" layer="95" xref="yes"/>
-</segment>
 <segment>
 <pinref part="JP10" gate="A" pin="2"/>
@@
 <junction x="238.76" y="93.98"/>
 </segment>
-</net>
+<segment>
+<pinref part="IC2" gate="G$1" pin="VOUT"/>
+<wire x1="294.64" y1="86.36" x2="284.48" y2="86.36" width="0.1524" layer="91"/>
+<label x="284.48" y="86.36" size="1.778" layer="95" rot="R180" xref="yes"/>
+</segment>
+</net>

Commit message: Add files via upload
Parts:
- removed R11, R12: (no value), resistor:R-US_0207/7
- added R3, R6: (no value), resistor:R-US_0207/7
- renumbered JP10 to JP7, JP15 to JP2, JP16 to JP8, JP17 to JP1, JP18 to JP9, JP28 to JP6, JP29 to JP5, JP30 to JP4, R10 to R2
Connections:
- net +5V_UNO: now also R6.1; no longer R8.1
- net ACTION_BUTTON: now also R5.2; no longer R12.2
- net GND: now also R3.1, R8.1; no longer R11.1, R12.1
- net N$8: now also R8.2; no longer R5.2
- net PLAYLIVE_SWITCH: now also R3.2; no longer R9.2
- net PLAYRECORDING_SWITCH: now also R4.2; no longer R11.2
- net RESET_BUTTON: now also R9.2; no longer R4.2
- net SCL: now also R7.2; no longer R8.2
- net SDA: now also R6.2; no longer R7.2
Other:
- moved on the sheet: R4, R5, R7, R8, R9
